Commit message: aulas

File: Aula12/p_tfonte_description/urdf/p_tfonte.gazebo.xacro (robot description, xacro)
@@ -5,5 +5,5 @@
   <xacro:arg name="imu_visual"    default="false"/>
   <gazebo reference="base_link">
-    <material>Gazebo/DarkGrey</material>
+    <material>Gazebo/Yellow</material>
   </gazebo>
   <gazebo reference="wheel_left_link">
