Commit message: aulas

File: Aula14/p_teamhunt_description_prep/urdf/p_teamhunt.gazebo.xacro (robot description, xacro)
@@ -168,3 +168,16 @@
     </sensor>
   </gazebo>
+  <gazebo reference="base_link">
+    <sensor name="base_link" type="contact">
+      <update_rate>1000.0</update_rate>
+      <always_on>true</always_on>
+      <contact>
+        <collision> "base_footprint_fixed_joint_lump__base_link_collision" </collision>
+      </contact>
+      <plugin name="base_link_contact_sensor_plugin" filename="libgazebo_ros_bumper.so">
+        <bumperTopicName>contact</bumperTopicName>
+        <frameName>world</frameName>
+      </plugin>
+    </sensor>
+  </gazebo>
 </robot>
